File: Keyboard PCB/Keyboard PCB.kicad_sch (KiCad schematic)
At the start: 0 parts

Commit message: Made the Schematic
Parts:
- added D1, D2: SK6812MINI-E, symbol SK6812MINI-E:SK6812MINI-E
- added SW1, SW2, SW3, SW4, SW5, SW6: SW_Push, Button_Switch_Keyboard:SW_Cherry_MX_1.00u_PCB, symbol Switch:SW_Push
- added U1: MOUDLE-SEEEDUINO-XIAO, symbol XIAO_RP2040:MOUDLE-SEEEDUINO-XIAO
Connections:
- new net: D1.1 (DOUT), D2.4 (DIN)
- new net: D1.4 (DIN), U1.5 (PA8_A4_D4_SDA)
- new net: SW5.1, U1.7 (PB08_A6_D6_TX)
- new net: SW4.1, U1.8 (PB09_A7_D7_RX)
- new net: SW2.1, U1.10 (PA5_A9_D9_MISO)
- new net: SW3.1, U1.9 (PA7_A8_D8_SCK)
- new net: SW6.1, U1.6 (PA9_A5_D5_SCL)
- new net: SW1.1, U1.11 (PA6_A10_D10_MOSI)
- new net +5V: D1.1 (DOUT), D2.1 (DOUT)
- new net GND: D1.3 (VSS), D2.3 (VSS), SW1.2, SW2.2, SW3.2, SW4.2, SW5.2, SW6.2, U1.13 (GND)
