File: Keyboard PCB/_autosave-Keyboard PCB.kicad_pcb (KiCad board)
At the start: 2 copper layers, 3.6 x 3.3 mm, 9 parts, among them SW1 SW_Push, SW2 SW_Push, SW3 SW_Push, SW4 SW_Push, SW5 SW_Push, SW6 SW_Push, U1 MOUDLE-SEEEDUINO-XIAO

Commit message: PCB (first revision)
Parts:
- D1, D2: value SK6812MINI-E -> SK6812MINI; footprint footprints:SK6812MINI-E_fixed -> LED_SMD:LED_SK6812MINI_PLCC4_3.5x3.5mm_P1.75mm
- moved D2 38.7 mm to (32.7, 58.7)
- moved D1 37.5 mm to (70.8, 58.7)
- moved SW5 4.76 mm to (102.6, 54.5)
- moved SW6 4.76 mm to (102.6, 73.5)
- moved U1 2.87 mm to (76.2, 42.9)
Connections:
- D1 pad 1: +5V -> Net-(D1-DOUT)
- D1 pad 2: (no net) -> GND
- D1 pad 3: GND -> Net-(D1-DIN)
- D1 pad 4: Net-(D1-DIN) -> +5V
- D2 pad 1: +5V -> unconnected-(D2-DOUT-Pad1)
- D2 pad 2: (no net) -> GND
- D2 pad 3: GND -> Net-(D1-DOUT)
- D2 pad 4: Net-(D1-DOUT) -> +5V
Routing:
- net GND: track 0.00 -> 176.9 mm
- net Net-(U1-PA6_A10_D10_MOSI): track 0.00 -> 74.6 mm
- net Net-(U1-PA9_A5_D5_SCL): track 0.00 -> 47.8 mm
- net Net-(D1-DOUT): track 0.00 -> 39.3 mm
- net +5V: track 0.00 -> 39.2 mm
- net Net-(U1-PA5_A9_D9_MISO): track 0.00 -> 34.4 mm
- net Net-(U1-PB08_A6_D6_TX): track 0.00 -> 25.5 mm
- net Net-(U1-PB09_A7_D7_RX): track 0.00 -> 25.3 mm
- net Net-(D1-DIN): track 0.00 -> 22.6 mm
- net Net-(U1-PA7_A8_D8_SCK): track 0.00 -> 16.3 mm
Other:
- board outline removed

Commit message: Updated PCB
Parts:
- moved U1 2.38 mm to (76.2, 45.2)
Routing:
- net Net-(U1-PB08_A6_D6_TX): track 25.5 -> 19.4 mm
- net Net-(U1-PA9_A5_D5_SCL): track 47.8 -> 42.3 mm
- net GND: track 176.9 -> 172.5 mm
- net Net-(U1-PB09_A7_D7_RX): track 25.3 -> 27.4 mm
- net Net-(D1-DIN): track 22.6 -> 20.7 mm
- net Net-(U1-PA7_A8_D8_SCK): track 16.3 -> 15.4 mm
- net unconnected-(U1-5V-Pad14): track 0.00 -> 0.64 mm
Other:
- board outline added: 85.7 x 53.4 mm
Changed lines of the file:
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@@
 	(footprint "footprints:XIAO-Generic-Hybrid-14P-2.54-21X17.8MM"
 		(layer "B.Cu")
-		(at 76.2 42.8625 180)
+		(at 76.2 45.24375 180)
 		(property "Reference" "U1"
 			(at -0.48125 -4.73875 0)
@@
 		(embedded_fonts no)
 	)
+	(gr_rect
+		(start 23.8125 34.71875)
+		(end 109.5375 88.10625)
+		(stroke
+			(width 0.05)
+			(type default)
+		)
+		(fill no)
+		(layer "Edge.Cuts")
+	)
 	(segment
-		(start 67.6275 76.04125)
-		(end 67.6275 60.96)
+		(start 68.8925 40.48125)
+		(end 68.575 40.16375)
 		(width 0.2)
 		(layer "F.Cu")
@@
 	)
 	(segment
-		(start 96.2025 56.99125)
-		(end 95.40875 56.99125)
+		(start 67.6275 76.04125)
+		(end 67.6275 60.96)
 		(width 0.2)
 		(layer "F.Cu")
@@
 	)
 	(segment
-		(start 70.08025 58.50725)
-		(end 73.65725 58.50725)
+		(start 96.2025 56.99125)
+		(end 81.68835 56.99125)
 		(width 0.2)
 		(layer "F.Cu")
@@
 	)
 	(segment
+		(start 81.68835 56.99125)
+		(end 78.42235 60.25725)
+		(width 0.2)
+		(layer "F.Cu")
+		(net 1)
+	)
+	(segment
 		(start 67.6275 60.96)
 		(end 69.05625 59.53125)
@@
 	)
 	(segment
-		(start 73.65725 43.50475)
-		(end 68.575 38.4225)
+		(start 30.95625 74.6125)
+		(end 30.95625 59.53125)
 		(width 0.2)
 		(layer "F.Cu")
@@
 	)
 	(segment
-		(start 69.05625 59.53125)
-		(end 70.08025 58.50725)
+		(start 73.65725 40.48125)
+		(end 68.8925 40.48125)
 		(width 0.2)
 		(layer "F.Cu")
@@
 	)
 	(segment
-		(start 68.575 38.4225)
-		(end 68.575 37.7825)
+		(start 96.2025 76.04125)
+		(end 96.2025 56.99125)
 		(width 0.2)
 		(layer "F.Cu")
@@
 	)
 	(segment
-		(start 30.95625 74.6125)
-		(end 30.95625 59.53125)
+		(start 73.65725 58.50725)
+		(end 73.65725 40.48125)
 		(width 0.2)
 		(layer "F.Cu")
@@
 	)
 	(segment
-		(start 96.2025 76.04125)
-		(end 96.2025 56.99125)
+		(start 70.08025 58.50725)
+		(end 73.65725 58.50725)
+		(width 0.2)
+		(layer "F.Cu")
+		(net 1)
+	)
+	(segment
+		(start 69.05625 59.53125)
+		(end 70.08025 58.50725)
 		(width 0.2)
 		(layer "F.Cu")
@@
 	)
 	(segment
-		(start 96.90525 60.25725)
+		(start 78.42235 60.25725)
 		(end 69.78225 60.25725)
 		(width 0.2)
@@
 	)
 	(segment
-		(start 95.40875 56.99125)
-		(end 92.14275 60.25725)
-		(width 0.2)
-		(layer "F.Cu")
-		(net 1)
-	)
-	(segment
-		(start 73.65725 58.50725)
-		(end 73.65725 43.50475)
+		(start 73.81875 59.53125)
+		(end 74.13625 59.53125)
 		(width 0.2)
 		(layer "F.Cu")
-		(net 1)
+		(net 2)
 	)
 	(segment
-		(start 80.9625 48.265)
-		(end 83.825 45.4025)
+		(start 72.55625 59.53125)
+		(end 73.81875 59.53125)
 		(width 0.2)
 		(layer "F.Cu")
@@
 	)
 	(segment
-		(start 73.81875 59.53125)
-		(end 74.13625 59.53125)
+		(start 80.9625 50.64625)
+		(end 83.825 47.78375)
 		(width 0.2)
 		(layer "F.Cu")
@@
 	)
 	(segment
-		(start 80.9625 57.15)
-		(end 80.9625 48.265)
+		(start 78.58125 59.53125)
+		(end 80.9625 57.15)
 		(width 0.2)
 		(layer "F.Cu")
@@
 	)
 	(segment
-		(start 72.55625 59.53125)
-		(end 73.81875 59.53125)
+		(start 84.1425 47.625)
+		(end 83.825 47.9425)
 		(width 0.2)
 		(layer "F.Cu")
@@
 	)
 	(segment
-		(start 78.58125 59.53125)
-		(end 80.9625 57.15)
+		(start 73.81875 59.53125)
+		(end 78.58125 59.53125)
 		(width 0.2)
 		(layer "F.Cu")
@@
 	)
 	(segment
-		(start 73.81875 59.53125)
-		(end 78.58125 59.53125)
+		(start 80.9625 57.15)
+		(end 80.9625 50.64625)
 		(width 0.2)
 		(layer "F.Cu")
@@
 	)
 	(segment
-		(start 28.1265 76.621564)
-		(end 28.1265 58.784)
+		(start 28.1265 58.784)
+		(end 41.66675 45.24375)
 		(width 0.2)
 		(layer "F.Cu")
@@
 	)
 	(segment
-		(start 28.947186 77.44225)
-		(end 28.1265 76.621564)
+		(start 30.107814 77.44225)
+		(end 28.947186 77.44225)
 		(width 0.2)
 		(layer "F.Cu")
@@
 	)
 	(segment
-		(start 44.048 42.8625)
-		(end 68.575 42.8625)
+		(start 28.1265 76.621564)
+		(end 28.1265 58.784)
 		(width 0.2)
 		(layer "F.Cu")
@@
 	)
 	(segment
-		(start 28.1265 58.784)
-		(end 44.048 42.8625)
+		(start 28.947186 77.44225)
+		(end 28.1265 76.621564)
 		(width 0.2)
 		(layer "F.Cu")
@@
 	)
 	(segment
-		(start 30.107814 77.44225)
-		(end 28.947186 77.44225)
+		(start 41.66675 45.24375)
+		(end 68.575 45.24375)
 		(width 0.2)
 		(layer "F.Cu")
@@
 	)
 	(segment
+		(start 67.53724 45.4025)
+		(end 68.575 45.4025)
+		(width 0.2)
+		(layer "B.Cu")
+		(net 5)
+	)
+	(segment
+		(start 54.9275 58.01224)
+		(end 66.30699 46.63275)
+		(width 0.2)
+		(layer "B.Cu")
+		(net 6)
+	)
+	(segment
 		(start 54.9275 73.50125)
 		(end 54.9275 58.01224)
@@
 	)
 	(segment
-		(start 54.9275 58.01224)
-		(end 67.53724 45.4025)
+		(start 66.30699 46.63275)
+		(end 67.424 46.63275)
 		(width 0.2)
 		(layer "B.Cu")
@@
 	)
 	(segment
-		(start 67.53724 45.4025)
-		(end 68.575 45.4025)
+		(start 67.424 46.63275)
+		(end 68.575 47.78375)
 		(width 0.2)
 		(layer "B.Cu")
@@
 	(segment
 		(start 54.9275 54.45125)
-		(end 61.43625 47.9425)
+		(end 59.055 50.32375)
 		(width 0.2)
 		(layer "F.Cu")
@@
 	)
 	(segment
-		(start 61.43625 47.9425)
-		(end 68.575 47.9425)
+		(start 59.055 50.32375)
+		(end 68.575 50.32375)
 		(width 0.2)
 		(layer "F.Cu")
@@
 	)
 	(segment
-		(start 73.9775 55.885)
-		(end 68.575 50.4825)
+		(start 71.59625 55.885)
+		(end 68.575 52.86375)
+		(width 0.2)
+		(layer "B.Cu")
+		(net 8)
+	)
+	(segment
+		(start 76.2 71.27875)
+		(end 76.2 55.885)
 		(width 0.2)
 		(layer "B.Cu")
@@
 	(segment
 		(start 73.9775 73.50125)
-		(end 73.9775 55.885)
+		(end 76.2 71.27875)
 		(width 0.2)
 		(layer "B.Cu")
@@
 	)
 	(segment
-		(start 107.315 54.45125)
-		(end 87.15375 54.45125)
+		(start 76.2 55.885)
+		(end 71.59625 55.885)
 		(width 0.2)
-		(layer "F.Cu")
-		(net 9)
+		(layer "B.Cu")
+		(net 8)
 	)
 	(segment
-		(start 83.825 51.1225)
-		(end 83.825 50.4825)
+		(start 102.5525 54.45125)
+		(end 85.4125 54.45125)
 		(width 0.2)
 		(layer "F.Cu")
@@
 	)
 	(segment
-		(start 87.15375 54.45125)
-		(end 83.825 51.1225)
+		(start 85.4125 54.45125)
+		(end 83.825 52.86375)
 		(width 0.2)
 		(layer "F.Cu")
@@
 	)
 	(segment
-		(start 103.9535 55.031564)
-		(end 103.9535 53.870936)
+		(start 84.23574 54.85225)
+		(end 82.724 53.34051)
 		(width 0.2)
 		(layer "F.Cu")
@@
 	)
 	(segment
-		(start 103.9535 53.870936)
-		(end 100.565064 50.4825)
+		(start 102.5525 56.432564)
+		(end 100.972186 54.85225)
 		(width 0.2)
 		(layer "F.Cu")
@@
 	)
 	(segment
-		(start 102.946314 50.4825)
-		(end 90.96375 50.4825)
+		(start 82.724 51.42475)
+		(end 83.825 50.32375)
 		(width 0.2)
 		(layer "F.Cu")
@@
 	)
 	(segment
-		(start 102.5525 56.432564)
-		(end 103.9535 55.031564)
+		(start 100.972186 54.85225)
+		(end 84.23574 54.85225)
 		(width 0.2)
 		(layer "F.Cu")
@@
 	)
 	(segment
-		(start 93.345 50.4825)
-		(end 90.4875 47.625)
+		(start 83.825 51.1225)
+		(end 83.825 50.4825)
 		(width 0.2)
 		(layer "F.Cu")
@@
 	)
 	(segment
-		(start 84.1425 47.625)
-		(end 83.825 47.9425)
+		(start 82.724 53.34051)
+		(end 82.724 51.42475)
 		(width 0.2)
 		(layer "F.Cu")
@@
 	)
 	(segment
-		(start 90.4875 47.625)
-		(end 84.1425 47.625)
+		(start 68.575 38.4225)
+		(end 68.575 37.7825)
 		(width 0.2)
 		(layer "F.Cu")
-		(net 10)
+		(net 11)
 	)
 	(embedded_fonts no)
